File: LoRa/_saved_LoRa_PMOD.sch (KiCad schematic (older format))
At the start: 5 parts, among them P1 PMOD_LoRa, P3 Extension, U1 RFM95W-868S2

Commit message: New version
Parts:
- removed P3: Extension, Pin_Headers:Pin_Header_Straight_1x05, symbol CONN_01X05
- added P2: Ext, Pin_Headers:Pin_Header_Straight_1x03_Pitch2.00mm, symbol CONN_01X03
- AE1: footprint Connectors:SMA_THT_Jack_Straight -> Connectors:SMB_Straight
Connections:
- net DIO3: now also P2.3 (P3)
- net DIO4: now also P2.2 (P2)
- net DIO5: now also P2.1 (P1)
Changed lines of the file:
@@
 Wire Wire Line
 	5700 5050 5800 5050
-$Comp
-L CONN_01X05 P3
-U 1 1 5BFAAF2D
-P 2850 5850
-F 0 "P3" H 2850 6150 50  0000 C CNN
-F 1 "Extension" V 2950 5850 50  0000 C CNN
-F 2 "Pin_Headers:Pin_Header_Straight_1x05" H 2850 5850 50  0001 C CNN
-F 3 "" H 2850 5850 50  0000 C CNN
-	1    2850 5850
-	-1   0    0    1
-$EndComp
 Text GLabel 4200 5550 0    60   Input ~ 0
 DIO3
@@
 Wire Wire Line
 	4200 5650 4300 5650
-Text GLabel 3150 5650 2    60   Input ~ 0
-VCC
-Text GLabel 3150 5750 2    60   Input ~ 0
-GND
 Text GLabel 3150 6050 2    60   Input ~ 0
 DIO5
@@
 	5700 5250 5800 5250
 Wire Wire Line
-	3050 5650 3150 5650
+	2900 5850 3150 5850
 Wire Wire Line
-	3050 5750 3150 5750
+	2900 5950 3150 5950
 Wire Wire Line
-	3050 5850 3150 5850
-Wire Wire Line
-	3050 5950 3150 5950
-Wire Wire Line
-	3050 6050 3150 6050
+	2900 6050 3150 6050
 Wire Wire Line
 	3550 3850 3550 3750
@@
 F 0 "AE1" H 6425 4475 50  0000 R CNN
 F 1 "Ant" H 6425 4400 50  0000 R CNN
-F 2 "Connectors:SMA_THT_Jack_Straight" H 6500 4400 50  0001 C CNN
+F 2 "Connectors:SMB_Straight" H 6500 4400 50  0001 C CNN
 F 3 "" H 6500 4400 50  0001 C CNN
 	1    6500 4300
@@
 Wire Wire Line
 	6500 4500 6500 4600
+$Comp
+L CONN_01X03 P2
+U 1 1 5BFB07D0
+P 2700 5950
+F 0 "P2" H 2700 6150 50  0000 C CNN
+F 1 "Ext" V 2800 5950 50  0000 C CNN
+F 2 "Pin_Headers:Pin_Header_Straight_1x03_Pitch2.00mm" H 2700 5950 50  0001 C CNN
+F 3 "" H 2700 5950 50  0000 C CNN
+	1    2700 5950
+	-1   0    0    1
+$EndComp
 $EndSCHEMATC
