File: LoRa/LoRa_PMOD.sch (KiCad schematic (older format))
At the start: 5 parts, among them P1 PMOD_LoRa, P2 Antenna, P3 Extension, U1 RFM95W-868S2

Commit message: Fixing 3D model
Parts:
- C1: footprint (none) -> Capacitors_SMD:C_0805_HandSoldering
- P1: footprint (none) -> Pin_Headers:Pin_Header_Angled_2x06
- P2: footprint (none) -> Pin_Headers:Pin_Header_Straight_1x02
- P3: footprint (none) -> Pin_Headers:Pin_Header_Straight_1x05
- U1: footprint XCVR_RFM95W-868S2 -> RFM95W-868S2:XCVR_RFM95W-868S2
Changed lines of the file:
@@
 LIBS:valves
 LIBS:RFM95W-868S2
+LIBS:radiona
+LIBS:LoRa_PMOD-cache
 EELAYER 25 0
 EELAYER END
@@
 F 0 "P1" H 4900 4550 50  0000 C CNN
 F 1 "PMOD_LoRa" H 4900 3850 50  0000 C CNN
-F 2 "" H 4900 3000 50  0000 C CNN
+F 2 "Pin_Headers:Pin_Header_Angled_2x06" H 4900 3000 50  0001 C CNN
 F 3 "" H 4900 3000 50  0000 C CNN
 	1    4900 4200
@@
 F 0 "C1" H 3575 4100 50  0000 L CNN
 F 1 "C1" H 3575 3900 50  0000 L CNN
-F 2 "" H 3588 3850 50  0000 C CNN
+F 2 "Capacitors_SMD:C_0805_HandSoldering" H 3588 3850 50  0001 C CNN
 F 3 "" H 3550 4000 50  0000 C CNN
 	1    3550 4000
@@
 F 0 "U1" H 4399 6001 50  0000 L BNN
 F 1 "RFM95W-868S2" H 4399 4749 50  0000 L BNN
-F 2 "XCVR_RFM95W-868S2" H 5000 5450 50  0001 L BNN
+F 2 "RFM95W-868S2:XCVR_RFM95W-868S2" H 5000 5450 50  0001 L BNN
 F 3 "" H 5000 5450 50  0001 L BNN
 F 4 "Unavailable" H 5000 5450 50  0001 L BNN "Field4"
@@
 F 0 "P3" H 2850 6150 50  0000 C CNN
 F 1 "Extension" V 2950 5850 50  0000 C CNN
-F 2 "" H 2850 5850 50  0000 C CNN
+F 2 "Pin_Headers:Pin_Header_Straight_1x05" H 2850 5850 50  0001 C CNN
 F 3 "" H 2850 5850 50  0000 C CNN
 	1    2850 5850
@@
 F 0 "P2" H 2850 5500 50  0000 C CNN
 F 1 "Antenna" V 2950 5350 50  0000 C CNN
-F 2 "" H 2850 5350 50  0000 C CNN
+F 2 "Pin_Headers:Pin_Header_Straight_1x02" H 2850 5350 50  0001 C CNN
 F 3 "" H 2850 5350 50  0000 C CNN
 	1    2850 5350
@@
 Wire Wire Line
 	5700 5750 5800 5750
+$Comp
+L LOGO #G1
+U 1 1 5BFAC680
+P 3450 2200
+F 0 "#G1" H 3450 2080 60  0001 C CNN
+F 1 "LOGO" H 3450 2320 60  0001 C CNN
+F 2 "" H 3450 2200 60  0001 C CNN
+F 3 "" H 3450 2200 60  0001 C CNN
+	1    3450 2200
+	1    0    0    -1
+$EndComp
 $EndSCHEMATC

Commit message: Fixing PMOD pinout
Connections:
- net +3V3: now also P1.1 (P1), P1.2 (P2); no longer P1.12 (P12), P1.6 (P6)
- net CS: now also P1.11 (P11); no longer P1.1 (P1)
- net DIO0: now also P1.12 (P12); no longer P1.7 (P7)
- net DIO1: now also P1.8 (P8); no longer P1.9 (P9)
- net DIO2: now also P1.6 (P6); no longer P1.10 (P10)
- net GND: now also P1.3 (P3), P1.4 (P4); no longer P1.11 (P11), P1.5 (P5)
- net MISO: now also P1.7 (P7); no longer P1.3 (P3)
- net MOSI: now also P1.9 (P9); no longer P1.2 (P2)
- net RESET: now also P1.10 (P10); no longer P1.8 (P8)
- net SCK: now also P1.5 (P5); no longer P1.4 (P4)
Changed lines of the file:
@@
 	1    0    0    -1
 $EndComp
+Text GLabel 4550 4450 0    60   Input ~ 0
+CS
+Text GLabel 4550 4250 0    60   Input ~ 0
+MISO
+Text GLabel 5250 4050 2    60   Input ~ 0
+GND
+Text GLabel 5250 4450 2    60   Input ~ 0
+DIO0
+Text GLabel 5250 4250 2    60   Input ~ 0
+DIO1
+Text GLabel 4550 4050 0    60   Input ~ 0
+GND
+Text GLabel 4550 4350 0    60   Input ~ 0
+MOSI
+Text GLabel 4550 4150 0    60   Input ~ 0
+SCK
 Text GLabel 4550 3950 0    60   Input ~ 0
-CS
-Text GLabel 4550 4050 0    60   Input ~ 0
-MISO
-Text GLabel 4550 4150 0    60   Input ~ 0
-GND
-Text GLabel 4550 4250 0    60   Input ~ 0
-DIO0
-Text GLabel 4550 4350 0    60   Input ~ 0
-DIO1
-Text GLabel 4550 4450 0    60   Input ~ 0
-GND
+VCC
+Text GLabel 5250 4350 2    60   Input ~ 0
+RESET
+Text GLabel 5250 4150 2    60   Input ~ 0
+DIO2
 Text GLabel 5250 3950 2    60   Input ~ 0
-MOSI
-Text GLabel 5250 4050 2    60   Input ~ 0
-SCK
-Text GLabel 5250 4150 2    60   Input ~ 0
-VCC
-Text GLabel 5250 4250 2    60   Input ~ 0
-RESET
-Text GLabel 5250 4350 2    60   Input ~ 0
-DIO2
-Text GLabel 5250 4450 2    60   Input ~ 0
-VCC
-Wire Wire Line
-	4550 3950 4650 3950
-Wire Wire Line
-	4550 4050 4650 4050
-Wire Wire Line
-	4550 4150 4650 4150
-Wire Wire Line
-	4550 4450 4650 4450
-Wire Wire Line
-	5150 3950 5250 3950
-Wire Wire Line
-	5150 4050 5250 4050
-Wire Wire Line
-	5150 4150 5250 4150
-Wire Wire Line
-	5150 4250 5250 4250
-Wire Wire Line
-	5150 4450 5250 4450
-Wire Wire Line
-	4550 4250 4650 4250
-Wire Wire Line
-	4550 4350 4650 4350
-Wire Wire Line
-	5150 4350 5250 4350
+VCC
 $Comp
 L +3.3V #PWR01
@@
 	1    0    0    -1
 $EndComp
+Wire Wire Line
+	4550 3950 4650 3950
+Wire Wire Line
+	4550 4050 4650 4050
+Wire Wire Line
+	5150 3950 5250 3950
+Wire Wire Line
+	5150 4050 5250 4050
+Wire Wire Line
+	5150 4150 5250 4150
+Wire Wire Line
+	4550 4150 4650 4150
+Wire Wire Line
+	4550 4250 4650 4250
+Wire Wire Line
+	4550 4350 4650 4350
+Wire Wire Line
+	4550 4450 4650 4450
+Wire Wire Line
+	5150 4450 5250 4450
+Wire Wire Line
+	5150 4350 5250 4350
+Wire Wire Line
+	5150 4250 5250 4250
 $EndSCHEMATC

Commit message: New version
Parts:
- removed P2: Antenna, Pin_Headers:Pin_Header_Straight_1x02, symbol CONN_01X02
- removed P3: Extension, Pin_Headers:Pin_Header_Straight_1x05, symbol CONN_01X05
- added AE1: Ant, Connectors:SMA_THT_Jack_Straight, symbol Antenna_Shield
- added P?: Ext, symbol CONN_01X03
Connections:
- net ANT: now also AE1.1 (A)
- net DIO3: now also P?.3 (P3)
- net DIO4: now also P?.2 (P2)
- net DIO5: now also P?.1 (P1)
- net GND: now also AE1.2 (Shield)
Changed lines of the file:
@@
 Wire Wire Line
 	5700 5050 5800 5050
-$Comp
-L CONN_01X05 P3
-U 1 1 5BFAAF2D
-P 2850 5850
-F 0 "P3" H 2850 6150 50  0000 C CNN
-F 1 "Extension" V 2950 5850 50  0000 C CNN
-F 2 "Pin_Headers:Pin_Header_Straight_1x05" H 2850 5850 50  0001 C CNN
-F 3 "" H 2850 5850 50  0000 C CNN
-	1    2850 5850
-	-1   0    0    1
-$EndComp
 Text GLabel 4200 5550 0    60   Input ~ 0
 DIO3
@@
 Wire Wire Line
 	4200 5650 4300 5650
-$Comp
-L CONN_01X02 P2
-U 1 1 5BFAB036
-P 2850 5350
-F 0 "P2" H 2850 5500 50  0000 C CNN
-F 1 "Antenna" V 2950 5350 50  0000 C CNN
-F 2 "Pin_Headers:Pin_Header_Straight_1x02" H 2850 5350 50  0001 C CNN
-F 3 "" H 2850 5350 50  0000 C CNN
-	1    2850 5350
-	-1   0    0    1
-$EndComp
-Text GLabel 3150 5650 2    60   Input ~ 0
-VCC
-Text GLabel 3150 5750 2    60   Input ~ 0
-GND
 Text GLabel 3150 6050 2    60   Input ~ 0
 DIO5
@@
 Text GLabel 3150 5850 2    60   Input ~ 0
 DIO3
-Text GLabel 3150 5400 2    60   Input ~ 0
-GND
 Text GLabel 5800 5250 2    60   Input ~ 0
 ANT
@@
 	5700 5250 5800 5250
 Wire Wire Line
-	3050 5400 3150 5400
+	2900 5850 3150 5850
 Wire Wire Line
-	3050 5650 3150 5650
+	2900 5950 3150 5950
 Wire Wire Line
-	3050 5750 3150 5750
-Wire Wire Line
-	3050 5850 3150 5850
-Wire Wire Line
-	3050 5950 3150 5950
-Wire Wire Line
-	3050 6050 3150 6050
-Text GLabel 3150 5300 2    60   Input ~ 0
-ANT
-Wire Wire Line
-	3050 5300 3150 5300
+	2900 6050 3150 6050
 Wire Wire Line
 	3550 3850 3550 3750
@@
 Wire Wire Line
 	5150 4250 5250 4250
+$Comp
+L Antenna_Shield AE1
+U 1 1 5BFB01E5
+P 6500 4300
+F 0 "AE1" H 6425 4475 50  0000 R CNN
+F 1 "Ant" H 6425 4400 50  0000 R CNN
+F 2 "Connectors:SMA_THT_Jack_Straight" H 6500 4400 50  0001 C CNN
+F 3 "" H 6500 4400 50  0001 C CNN
+	1    6500 4300
+	1    0    0    -1
+$EndComp
+Text GLabel 6600 4600 3    60   Input ~ 0
+GND
+Wire Wire Line
+	6600 4600 6600 4500
+Text GLabel 6500 4600 3    60   Input ~ 0
+ANT
+Wire Wire Line
+	6500 4500 6500 4600
+$Comp
+L CONN_01X03 P?
+U 1 1 5BFB07D0
+P 2700 5950
+F 0 "P?" H 2700 6150 50  0000 C CNN
+F 1 "Ext" V 2800 5950 50  0000 C CNN
+F 2 "" H 2700 5950 50  0000 C CNN
+F 3 "" H 2700 5950 50  0000 C CNN
+	1    2700 5950
+	-1   0    0    1
+$EndComp
 $EndSCHEMATC

Commit message: Changing sch
Parts:
- AE1: footprint Connectors:SMA_THT_Jack_Straight -> Connectors:SMB_Straight
- P2: renamed from P?; footprint (none) -> Pin_Headers:Pin_Header_Straight_1x03_Pitch2.00mm
Changed lines of the file:
@@
 F 0 "AE1" H 6425 4475 50  0000 R CNN
 F 1 "Ant" H 6425 4400 50  0000 R CNN
-F 2 "Connectors:SMA_THT_Jack_Straight" H 6500 4400 50  0001 C CNN
+F 2 "Connectors:SMB_Straight" H 6500 4400 50  0001 C CNN
 F 3 "" H 6500 4400 50  0001 C CNN
 	1    6500 4300
@@
 	6500 4500 6500 4600
 $Comp
-L CONN_01X03 P?
+L CONN_01X03 P2
 U 1 1 5BFB07D0
 P 2700 5950
-F 0 "P?" H 2700 6150 50  0000 C CNN
+F 0 "P2" H 2700 6150 50  0000 C CNN
 F 1 "Ext" V 2800 5950 50  0000 C CNN
-F 2 "" H 2700 5950 50  0000 C CNN
+F 2 "Pin_Headers:Pin_Header_Straight_1x03_Pitch2.00mm" H 2700 5950 50  0001 C CNN
 F 3 "" H 2700 5950 50  0000 C CNN
 	1    2700 5950

Commit message: switching to kicad v5 - edcuts not working
Parts:
- AE1: symbol Antenna_Shield -> LoRa_PMOD-rescue:Antenna_Shield
- C1: symbol C -> LoRa_PMOD-rescue:C
- P1: symbol CONN_02X06 -> LoRa_PMOD-rescue:CONN_02X06
- P2: symbol CONN_01X03 -> LoRa_PMOD-rescue:CONN_01X03
- U1: symbol RFM95W-868S2 -> RFM95W-868S2:RFM95W-868S2
Changed lines of the file:
@@
-EESchema Schematic File Version 2
-LIBS:power
-LIBS:device
-LIBS:transistors
-LIBS:conn
-LIBS:linear
-LIBS:regul
-LIBS:74xx
-LIBS:cmos4000
-LIBS:adc-dac
-LIBS:memory
-LIBS:xilinx
-LIBS:microcontrollers
-LIBS:dsp
-LIBS:microchip
-LIBS:analog_switches
-LIBS:motorola
-LIBS:texas
-LIBS:intel
-LIBS:audio
-LIBS:interface
-LIBS:digital-audio
-LIBS:philips
-LIBS:display
-LIBS:cypress
-LIBS:siliconi
-LIBS:opto
-LIBS:atmel
-LIBS:contrib
-LIBS:valves
-LIBS:RFM95W-868S2
-LIBS:radiona
+EESchema Schematic File Version 4
 LIBS:LoRa_PMOD-cache
-EELAYER 25 0
+EELAYER 26 0
 EELAYER END
 $Descr A4 11693 8268
@@
 Pmod Interface Type 2A (expanded SPI)\n\n1	CS 	Out\n2	MOSI	Out\n3	MISO	In\n4	SCK		Out\n5	GND\n6	VCC\n7	GPIO	In/Out	InterfaceIn\n8	GPIO	In/Out	RESET 	Out\n9	GPIO	In/Out	CS2	Out\n10	GPIO	In/Out	CS3	Out\n11	GND	\n12	VCC
 $Comp
-L CONN_02X06 P1
+L LoRa_PMOD-rescue:CONN_02X06 P1
 U 1 1 5BFAA353
 P 4900 4200
@@
 VCC
 $Comp
-L +3.3V #PWR01
+L power:+3.3V #PWR01
 U 1 1 5BFAA7BB
 P 3550 3750
@@
 $EndComp
 $Comp
-L GND #PWR02
+L power:GND #PWR02
 U 1 1 5BFAA7D2
 P 3550 4250
@@
 $EndComp
 $Comp
-L +3.3V #PWR03
+L power:+3.3V #PWR03
 U 1 1 5BFAA7E7
 P 3100 3850
@@
 	3100 4100 3100 3850
 $Comp
-L C C1
+L LoRa_PMOD-rescue:C C1
 U 1 1 5BFAA809
 P 3550 4000
@@
 	3550 4150 3550 4250
 $Comp
-L RFM95W-868S2 U1
+L RFM95W-868S2:RFM95W-868S2 U1
 U 1 1 5BFAAA0A
 P 5000 5450
@@
 	5700 5750 5800 5750
 $Comp
-L LOGO #G1
+L radiona:LOGO #G1
 U 1 1 5BFAC680
 P 3450 2200
@@
 	5150 4250 5250 4250
 $Comp
-L Antenna_Shield AE1
+L LoRa_PMOD-rescue:Antenna_Shield AE1
 U 1 1 5BFB01E5
 P 6500 4300
@@
 	6500 4500 6500 4600
 $Comp
-L CONN_01X03 P2
+L LoRa_PMOD-rescue:CONN_01X03 P2
 U 1 1 5BFB07D0
 P 2700 5950

Commit message: Fixing pinouts and pictures
Parts:
- U1: symbol RFM95W-868S2:RFM95W-868S2 -> LoRa_PMOD-rescue:RFM95W-868S2-RFM95W-868S2
Changed lines of the file:
@@
 	3550 4150 3550 4250
 $Comp
-L RFM95W-868S2:RFM95W-868S2 U1
+L LoRa_PMOD-rescue:RFM95W-868S2-RFM95W-868S2 U1
 U 1 1 5BFAAA0A
 P 5000 5450
@@
 	5700 5750 5800 5750
 $Comp
-L radiona:LOGO #G1
+L LoRa_PMOD-rescue:LOGO-radiona #G1
 U 1 1 5BFAC680
 P 3450 2200
