File: OV7670/arduCam_RC522.kicad_pcb (KiCad board)
At the start: 2 copper layers, 23.2 x 50.8 mm, 7 parts, among them J1 OV7670, J2 PMOD1, J3 PMOD2, J4 PMOD1_EXT, J5 PMOD2_EXT, J6 EXT1, J7 EXT2

Commit message: Update PCB
Parts:
- moved J2 2.25 mm to (157.2, 55.8)
- moved J3 1.00 mm to (157.2, 86.5)
- moved J4 1.00 mm to (157.2, 71.0)
Routing:
- net D5: track 39.1 -> 78.0 mm
- net Net-(J4-Pad4): track 31.6 -> 17.6 mm, vias 0 -> 1
- net Net-(J5-Pad2): track 24.8 -> 17.9 mm
- net PWDN: track 30.0 -> 23.9 mm
- net GND: track 63.9 -> 57.8 mm, vias 0 -> 1
- net Net-(J4-Pad2): track 20.4 -> 24.9 mm
- net SIOD: track 40.8 -> 36.9 mm
- net D4: track 37.9 -> 34.6 mm, vias 0 -> 1
- net D7: track 35.2 -> 32.3 mm
- net VSYNC: track 37.5 -> 34.8 mm
- net SIOC: track 33.0 -> 30.7 mm
- net Net-(J5-Pad6): track 15.2 -> 17.3 mm, vias 1 -> 0
- net HREF: track 29.5 -> 27.6 mm
- net Net-(J4-Pad6): track 15.6 -> 17.5 mm
- net Net-(J4-Pad1): track 25.0 -> 23.2 mm
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- added copper zone on B.Cu, net GND
- added copper zone on F.Cu, net GND

Commit message: Adding in labels
Parts:
- added ?: LOGO, parts:shutleworth, F.Cu at (151.8, 76.8)
- added G***: LOGO, parts:radiona, B.Cu at (152.2, 77.0)
Other:
- board text added: "3V3"
- board text added: "D0"
- board text added: "D1"
- board text added: "D11"
- board text added: "D2"
- board text added: "D3"
- board text added: "D4"
- board text added: "D5"
- board text added: "D6"
- board text added: "D7"
- board text added: "GND"
- board text added: "HREF"
- board text added: "PCLK"
- board text added: "PWDN"
- board text added: "RESET"
- board text added: "SOIC"
- board text added: "SOID"
- board text added: "VSYNC"
- board text added: "XCLK"
