File: I2S_Audio/I2S_Audio.kicad_pcb (KiCad board)
At the start: 2 copper layers, 41.5 x 18.5 mm, 20 parts, among them J1 PMOD, J2 AudioJack3_Ground, U1 CS4344-CZZ

Commit message: New versions
Other:
- board size 41.5 x 18.5 mm -> 41 x 20 mm
