File: MAX31855/MAX31855.kicad_pcb (KiCad board)
At the start: 2 copper layers, 24.5 x 18.5 mm, 11 parts, among them J1 PMOD, J2 Probe, U1 MAX31855JASA

Commit message: New versions
Parts:
- moved J2 7.50 mm to (166.5, 83.8)
Routing:
- net Net-(C3-Pad2): track 23.3 -> 30.8 mm
- net Net-(C3-Pad1): track 24.2 -> 31.7 mm
- added copper zone on B.Cu, net GND
- added copper zone on F.Cu, net GND
Other:
- board size 24.5 x 18.5 mm -> 32 x 20 mm
Changed lines of the file:
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@@
   (general
     (thickness 1.6)
-    (drawings 9)
-    (tracks 106)
+    (drawings 13)
+    (tracks 107)
     (zones 0)
     (modules 11)
@@
   )
   (setup
-    (last_trace_width 1)
+    (last_trace_width 0.25)
     (user_trace_width 0.5)
     (user_trace_width 0.7)
@@
       (outputformat 1)
       (mirror false)
-      (drillshape 1)
+      (drillshape 0)
       (scaleselection 1)
-      (outputdirectory ""))
+      (outputdirectory "Gerber/"))
   )
   (net 0 "")
@@
   )
   (module Connectors_Terminal_Blocks:TerminalBlock_Pheonix_MPT-2.54mm_2pol (layer F.Cu)
-    (at 174 83.75 270)
+    (at 166.5 83.75 270)
     (descr "2-way 2.54mm pitch terminal block, Phoenix MPT series")
     (fp_text reference J2 (at 1.27 -4.50088 270) (layer F.SilkS)
@@
       (xy -4.516743 0.903446) (xy -4.504214 0.908711) (xy -4.502362 0.909053) (xy -4.503792 0.904278)) (layer B.SilkS) (width 0.01))
   )
-  (gr_line (start 195 94.5) (end 170.5 94.5) (layer Edge.Cuts) (width 0.15))
-  (gr_line (start 195 76) (end 195 94.5) (layer Edge.Cuts) (width 0.15))
-  (gr_line (start 170.5 76) (end 195 76) (layer Edge.Cuts) (width 0.15))
-  (gr_line (start 170.5 94.5) (end 170.5 76) (layer Edge.Cuts) (width 0.15))
+  (gr_line (start 166.75 95) (end 195 95) (layer Edge.Cuts) (width 0.15))
+  (gr_line (start 163 95) (end 163.25 95) (layer Edge.Cuts) (width 0.15))
+  (gr_arc (start 165 95) (end 166.75 95) (angle -180) (layer Edge.Cuts) (width 0.15))
+  (gr_line (start 166.75 75) (end 195 75) (layer Edge.Cuts) (width 0.15))
+  (gr_line (start 163.25 75) (end 163 75) (layer Edge.Cuts) (width 0.15))
+  (gr_arc (start 165 75) (end 163.25 75) (angle -180) (layer Edge.Cuts) (width 0.15))
+  (gr_line (start 195 95) (end 195 75) (layer Edge.Cuts) (width 0.15))
+  (gr_line (start 163 75) (end 163 95) (layer Edge.Cuts) (width 0.15))
   (gr_text CS (at 192.75 91.75 180) (layer B.SilkS)
     (effects (font (size 1 1) (thickness 0.2)) (justify mirror))
@@
   (segment (start 175.75 85.953492) (end 175.413492 86.29) (width 1) (layer B.Cu) (net 4))
   (segment (start 175.75 82) (end 175.75 85.953492) (width 1) (layer B.Cu) (net 4))
+  (segment (start 174 86.29) (end 166.5 86.29) (width 1) (layer B.Cu) (net 4))
   (segment (start 177.375 77.5) (end 181 77.5) (width 1) (layer F.Cu) (net 5))
   (via (at 181 77.5) (size 0.8) (drill 0.4) (layers F.Cu B.Cu) (net 5))
@@
   (segment (start 185.450009 79.822061) (end 183.885 81.38707) (width 1) (layer F.Cu) (net 5))
   (segment (start 186.25 79) (end 185.45001 79.79999) (width 1) (layer F.Cu) (net 5))
-  (segment (start 174 83.75) (end 175.99949 83.75) (width 1) (layer F.Cu) (net 5))
-  (segment (start 176.624072 79.249072) (end 176.125 78.75) (width 1) (layer F.Cu) (net 5))
-  (segment (start 175.99949 83.75) (end 176.950009 82.799481) (width 1) (layer F.Cu) (net 5))
-  (segment (start 176.950009 79.575009) (end 176.624072 79.249072) (width 1) (layer F.Cu) (net 5))
-  (segment (start 176.950009 82.799481) (end 176.950009 79.575009) (width 1) (layer F.Cu) (net 5))
+  (segment (start 174 83.75) (end 166.5 83.75) (width 1) (layer F.Cu) (net 5))
+  (segment (start 176.125 78.75) (end 176.950009 79.575009) (width 1) (layer F.Cu) (net 5))
+  (segment (start 176.950009 79.575009) (end 176.950009 82.799481) (width 1) (layer F.Cu) (net 5))
+  (segment (start 176.950009 82.799481) (end 175.99949 83.75) (width 1) (layer F.Cu) (net 5))
+  (segment (start 175.99949 83.75) (end 174 83.75) (width 1) (layer F.Cu) (net 5))
   (segment (start 182.615 88.765002) (end 182.615 87.7) (width 1) (layer F.Cu) (net 6))
   (segment (start 183.024999 89.175001) (end 182.615 88.765002) (width 1) (layer F.Cu) (net 6))
@@
   (segment (start 181.345 86.634998) (end 183.899998 84.08) (width 1) (layer F.Cu) (net 8))
   (segment (start 181.345 87.7) (end 181.345 86.634998) (width 1) (layer F.Cu) (net 8))
+  (zone (net 1) (net_name GND) (layer F.Cu) (hatch edge 0.508)
+    (connect_pads (clearance 0.508))
+    (min_thickness 0.254)
+    (fill yes (arc_segments 16) (thermal_gap 0.508) (thermal_bridge_width 0.508))
+    (polygon
+      (pts
+        (xy 195 75) (xy 195 95) (xy 163 95) (xy 163 75)
+      )
+    )
+  )
+  (zone (net 1) (net_name GND) (layer B.Cu) (hatch edge 0.508)
+    (connect_pads (clearance 0.508))
+    (min_thickness 0.254)
+    (fill yes (arc_segments 16) (thermal_gap 0.508) (thermal_bridge_width 0.508))
+    (polygon
+      (pts
+        (xy 195 75) (xy 195 95) (xy 163 95) (xy 163 75)
+      )
+    )
+  )
 )
