File: PB9/PB9.kicad_pcb (KiCad board)
At the start: 2 copper layers, 31.2 x 21 mm, 7 parts, among them J1 PMOD_DB9, J2 DB9, J3 5V

Commit message: Fixing DB9
Parts:
- moved G*** 0.25 mm to (151.0, 76.2)
Changed lines of the file:
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@@
   (page A4)
   (layers
-    (0 F.Cu signal)
-    (31 B.Cu signal)
+    (0 F.Cu signal hide)
+    (31 B.Cu signal hide)
     (32 B.Adhes user)
     (33 F.Adhes user)
@@
   )
   (setup
-    (last_trace_width 0.5)
+    (last_trace_width 0.25)
     (user_trace_width 0.5)
     (user_trace_width 0.75)
@@
   )
   (module parts:radiona-12mm (layer B.Cu)
-    (at 151 76)
+    (at 151 76.25)
     (fp_text reference G*** (at 0 0) (layer B.SilkS) hide
       (effects (font (size 1.524 1.524) (thickness 0.3)) (justify mirror))
@@
       (xy -4.516743 0.903446) (xy -4.504214 0.908711) (xy -4.502362 0.909053) (xy -4.503792 0.904278)) (layer B.SilkS) (width 0.01))
   )
-  (gr_text 5V (at 162.5 86) (layer F.Mask)
+  (gr_text 5V (at 162.5 86) (layer F.SilkS)
     (effects (font (size 1.5 1.5) (thickness 0.3)))
   )
