File: ENC28J60/ENC28J60_PMOD/ENC28J60_PMOD.kicad_pcb (KiCad board)
At the start: 2 copper layers, 53.4 x 19.1 mm, 22 parts, among them J1 RJ45, J2 Conn_02x06_Odd_Even, U1 ENC28J60, Y1 Crystal

Commit message: Adding purple version
Parts:
- added G***: LOGO, parts:OSH_7x7, B.Cu at (149.9, 81.0)
