File: HDMI/HDMI.kicad_pcb (KiCad board)
At the start: 2 copper layers, 39.5 x 25.1 mm, 57 parts, among them J2 PMOD, P1 HDMI-D, U1 RN5RK501A, U2 PCA9306

Commit message: Fix #10 Fix #9 Fix #8
Parts:
- removed C10: 220nF, Capacitor_SMD:C_0603_1608Metric_Pad1.05x0.95mm_HandSolder
- removed G*** (x2): LOGO, parts2:radiona-10mm
- removed G***: LOGO, parts2:OSH_10x10
- removed G***: LOGO, parts2:shutleworth-12mm
- removed JP1, JP2, JP3, JP4, JP5, JP6: JUMP, Jumper:SolderJumper-2_P1.3mm_Bridged_RoundedPad1.0x1.5mm
- added D3: D_Zener_Small, Diode_SMD:D_SOD-323, F.Cu at (165.0, 59.4)
- added R28: 510, Resistor_SMD:R_0402_1005Metric, F.Cu at (133.5, 61.4)
- added R29: 4.7k, Resistor_SMD:R_0402_1005Metric, F.Cu at (126.7, 62.2)
- C1, C13, C2, C3, C4, C5, C6, C7, C8, C9: footprint Capacitor_SMD:C_0603_1608Metric_Pad1.05x0.95mm_HandSolder -> Capacitor_SMD:C_0402_1005Metric
- L1: footprint Inductor_SMD:L_1210_3225Metric_Pad1.42x2.65mm_HandSolder -> Inductor_SMD:L_1210_3225Metric
- R1, R10, R11, R12, R13, R14, R15, R16, R17, R18, R19, R2, R20, R21, R22, R23, R24, R25, R26, R27, R3, R4, R5, R6, R7, R8, R9: footprint Resistor_SMD:R_0603_1608Metric_Pad1.05x0.95mm_HandSolder -> Resistor_SMD:R_0402_1005Metric
- U1: footprint Package_TO_SOT_SMD:SOT-23-5_HandSoldering -> Package_TO_SOT_SMD:SOT-23-5
- U2: footprint Package_SO:SSOP-8_2.95x2.8mm_P0.65mm -> Package_SO:VSSOP-8_2.3x2mm_P0.5mm
Connections:
- C12 pad 1: Net-(C12-Pad1) -> +5V
- D1 pad 1: Net-(C12-Pad1) -> +5V
- R10 pad 1: Net-(JP2-Pad1) -> GPDI_D0+
- R11 pad 1: Net-(JP1-Pad2) -> +3V3
- R12 pad 1: Net-(JP1-Pad2) -> +3V3
- R13 pad 2: Net-(JP3-Pad1) -> GPDI_D1+
- R14 pad 1: Net-(JP3-Pad1) -> GPDI_D1+
- R15 pad 1: Net-(JP1-Pad2) -> +3V3
- R16 pad 1: Net-(JP1-Pad2) -> +3V3
- R17 pad 2: Net-(JP4-Pad1) -> GPDI_D2+
- R18 pad 1: Net-(JP4-Pad1) -> GPDI_D2+
- R19 pad 1: Net-(JP1-Pad2) -> +3V3
- R20 pad 1: Net-(JP1-Pad2) -> +3V3
- R21 pad 2: Net-(JP5-Pad1) -> GPDI_CLK+
- R22 pad 1: Net-(JP5-Pad1) -> GPDI_CLK+
- R23 pad 1: Net-(JP1-Pad2) -> +3V3
- R8 pad 1: Net-(JP1-Pad2) -> +3V3
- R9 pad 2: Net-(JP2-Pad1) -> GPDI_D0+
- U1 pad 1: Net-(C12-Pad1) -> LED_HDMI
- U1 pad 2: Net-(C12-Pad1) -> +5V
Routing:
- net GND: track 161.5 -> 0.00 mm, vias 18 -> 0
- net +5V: track 76.8 -> 0.00 mm, vias 4 -> 0
- net +3V3: track 68.6 -> 0.00 mm, vias 9 -> 0
- net GPDI_ETH+: track 42.6 -> 0.00 mm, vias 2 -> 0
- net GPDI_SCL: track 38.2 -> 0.00 mm, vias 4 -> 0
- net Net-(JP1-Pad2): track 37.6 -> 0.00 mm, vias 7 -> 0
- net PMOD_SCL: track 37.0 -> 0.00 mm, vias 1 -> 0
- net Net-(C13-Pad1): track 36.1 -> 0.00 mm, vias 8 -> 0
- net GPDI_ETH-: track 34.9 -> 0.00 mm
- net Net-(C12-Pad1): track 32.7 -> 0.00 mm, vias 2 -> 0
- net /CEC: track 32.2 -> 0.00 mm, vias 4 -> 0
- net GPDI_CLK+: track 28.8 -> 0.00 mm, vias 4 -> 0
- net GPDI_SDA: track 27.7 -> 0.00 mm, vias 2 -> 0
- net GPDI_D2+: track 25.0 -> 0.00 mm, vias 5 -> 0
- net LED_HDMI: track 22.2 -> 0.00 mm, vias 1 -> 0
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- removed copper zone on B.Cu, net GND
- removed copper zone on F.Cu, net GND
Other:
- copper layers 2 -> 4
