File: MIDI/midi.kicad_pcb (KiCad board)
At the start: 2 copper layers, 87 x 19.5 mm, 16 parts, among them J1 MIDI-IN, J2 MIDI_OUT, J3 MIDI-THROUGH, J4 PMOD, J5 EXT, U1 TLP2361

Commit message: Adding version number, adding gerber zip
Parts:
- moved G*** 11.1 mm to (71.5, 100.2)
Other:
- board text added: "V_1.0"
Changed lines of the file:
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@@
   (general
     (thickness 1.6)
-    (drawings 21)
+    (drawings 22)
     (tracks 262)
     (zones 0)
@@
   )
   (module MIDI:radiona-10mm (layer B.Cu)
-    (at 82.54 101.31 180)
+    (at 71.51 100.21 180)
     (fp_text reference G*** (at 0 0 180) (layer B.SilkS) hide
       (effects (font (size 1.524 1.524) (thickness 0.3)) (justify mirror))
@@
       (xy -4.18592 -1.25984) (xy -4.151381 -1.25984) (xy -4.130649 -1.261396)) (layer B.SilkS) (width 0.01))
   )
+  (gr_text V_1.0 (at 98.57 101.87) (layer B.SilkS)
+    (effects (font (size 1.5 1.5) (thickness 0.3)) (justify mirror))
+  )
   (gr_text +-2 (at 42.49 101.65) (layer B.SilkS)
