File: MIDI/midi.kicad_pcb (KiCad board)
At the start: 2 copper layers, 87 x 19.5 mm, 16 parts, among them J1 MIDI-IN, J2 MIDI_OUT, J3 MIDI-THROUGH, J4 PMOD, J5 EXT, U1 TLP2361

Commit message: Rerouting PCB - Adding logos
Parts:
- removed the G*** at (82.4, 90.7)
- removed the G*** at (60.8, 90.8)
- added REF**: OSHW-Logo2_7.3x6mm_SilkScreen, Symbol:OSHW-Logo2_7.3x6mm_SilkScreen, B.Cu at (61.0, 90.9)
- R1: value 220R -> 30R
- R2: value 220R -> 10R
- U1: footprint Package_SO:SO-6L_10x3.84mm_P1.27mm -> Package_SO:SO-6_4.4x3.6mm_P1.27mm
- moved G*** 14.2 mm to (82.3, 90.9)
- moved R5 7.65 mm to (96.3, 100.8)
Routing:
- net GND: track 166.7 -> 18.8 mm, vias 5 -> 27
- net Net-(D1-Pad1): track 21.3 -> 36.1 mm, vias 4 -> 5
- net +3V3: track 87.3 -> 94.1 mm, vias 0 -> 6
- net Net-(J1-Pad4): track 7.75 -> 2.88 mm
- net GN0: track 83.6 -> 81.4 mm, vias 2 -> 4
- net GP3: track 72.3 -> 74.0 mm, vias 1 -> 4
- net GP1: track 69.0 -> 70.2 mm
- net Net-(J3-Pad4): track 15.9 -> 17.1 mm, vias 0 -> 1
- net GN1: track 77.7 -> 76.7 mm
- net GN3: track 89.6 -> 90.6 mm
- net Net-(J2-Pad5): track 5.13 -> 6.03 mm, vias 0 -> 1
- net GP0: track 84.5 -> 85.4 mm
- net GN2: track 75.0 -> 75.7 mm
- net Net-(J3-Pad5): track 16.7 -> 17.4 mm, vias 1 -> 3
- net Net-(D1-Pad2): track 15.8 -> 15.7 mm, vias 2 -> 3
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Other:
- outline, holes or cut-outs redrawn
- board text added: "V_1.1"
- board text removed: "V_1.0"
