File: MIDI/midi.sch (KiCad schematic (older format))
At the start: 13 parts, among them J1 MIDI-IN, J2 MIDI_OUT, J3 MIDI-THROUGH, J4 PMOD, J5 EXT, U1 TLP2361

Commit message: Adding changes
Parts:
- U1: footprint Package_SO:SO-6L_10x3.84mm_P1.27mm -> Package_SO:SO-6_4.4x3.6mm_P1.27mm
Changed lines of the file:
@@
 F 0 "U1" H 3691 1946 50  0000 L CNN
 F 1 "TLP2361" H 3350 1550 50  0000 L CNN
-F 2 "Package_SO:SO-6L_10x3.84mm_P1.27mm" H 2550 1400 50  0001 L CIN
+F 2 "Package_SO:SO-6_4.4x3.6mm_P1.27mm" H 2550 1400 50  0001 L CIN
 F 3 "https://toshiba.semicon-storage.com/info/docget.jsp?did=29405&prodName=TLP2745" H 3142 1915 50  0001 L CNN
 	1    3250 1900

Commit message: Rerouting PCB - Adding logos
Parts:
- U1: Mouser (none) -> https://hr.mouser.com/ProductDetail/Toshiba/TLP2361TPLE/?qs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
Changed lines of the file:
@@
 F 2 "Package_SO:SO-6_4.4x3.6mm_P1.27mm" H 2550 1400 50  0001 L CIN
 F 3 "https://toshiba.semicon-storage.com/info/docget.jsp?did=29405&prodName=TLP2745" H 3142 1915 50  0001 L CNN
+F 4 "https://hr.mouser.com/ProductDetail/Toshiba/TLP2361TPLE/?qs=HVbQlW5zcXUn%252BfokbzIatg%3D%3D" H 3250 1900 50  0001 C CNN "Mouser"
 	1    3250 1900
 	1    0    0    -1
