File: VGA/VGA.sch (KiCad schematic (older format))
At the start: 20 parts, among them J1 DB15_Female_HighDensity, J2 VGA_PMOD

Commit message: Adding VGA V_1.0
Parts:
- added H1: MountingHole, MountingHole:MountingHole_3.5mm, symbol Mechanical:MountingHole
- J1: footprint (none) -> Connector_Dsub:DSUB-15-HD_Female_Horizontal_P2.29x1.98mm_EdgePinOffset3.03mm_Housed_MountingHolesOffset4.94mm
- J2: footprint (none) -> Connector_PinHeader_2.54mm:PinHeader_2x09_P2.54mm_Horizontal
- R1, R10, R11, R12, R13, R14, R15, R16, R17, R18, R2, R3, R4, R5, R6, R7, R8, R9: footprint (none) -> Resistor_SMD:R_0603_1608Metric
Connections:
- net B0: now also J2.18 (Pin_18); no longer J2.10 (Pin_10)
- net B1: now also J2.15 (Pin_15); no longer J2.9 (Pin_9)
- net B2: now also J2.14 (Pin_14); no longer J2.8 (Pin_8)
- net B3: now also J2.13 (Pin_13); no longer J2.7 (Pin_7)
- net G0: now also J2.17 (Pin_17); no longer J2.14 (Pin_14)
- net G1: now also J2.12 (Pin_12); no longer J2.13 (Pin_13)
- net G2: now also J2.11 (Pin_11); no longer J2.12 (Pin_12)
- net G3: now also J2.10 (Pin_10); no longer J2.11 (Pin_11)
- net R0: now also J2.16 (Pin_16); no longer J2.18 (Pin_18)
- net R1: now also J2.9 (Pin_9); no longer J2.17 (Pin_17)
- net R2: now also J2.8 (Pin_8); no longer J2.16 (Pin_16)
- net R3: now also J2.7 (Pin_7); no longer J2.15 (Pin_15)
Other:
- moved on the sheet: J2
