File: VGA/VGA.kicad_pcb (KiCad board)
At the start: 2 copper layers, 40.2 x 23 mm, 25 parts, among them J1 DB15_Female_HighDensity, J2 VGA_PMOD

Commit message: Connecting VGA connector to GND
Connections:
- J1 pad 0: (no net) -> GND
Other:
- board text added: "V_1.1"
- board text removed: "V_1.0"
Changed lines of the file:
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@@
     (mod_text_size 1 1)
     (mod_text_width 0.15)
-    (pad_size 1.524 1.524)
-    (pad_drill 0.762)
+    (pad_size 4 4)
+    (pad_drill 3.2)
     (pad_to_mask_clearance 0.051)
     (solder_mask_min_width 0.25)
@@
       (net 6 VSYNC))
     (pad 15 thru_hole circle (at -9.16 3.96 180) (size 1.6 1.6) (drill 1) (layers *.Cu *.Mask))
-    (pad 0 thru_hole circle (at -16.815 2.05 180) (size 4 4) (drill 3.2) (layers *.Cu *.Mask))
-    (pad 0 thru_hole circle (at 8.185 2.05 180) (size 4 4) (drill 3.2) (layers *.Cu *.Mask))
+    (pad 0 thru_hole circle (at -16.815 2.05 180) (size 4 4) (drill 3.2) (layers *.Cu *.Mask)
+      (net 4 GND))
+    (pad 0 thru_hole circle (at 8.185 2.05 180) (size 4 4) (drill 3.2) (layers *.Cu *.Mask)
+      (net 4 GND))
     (model /media/internal/FPGA/ulx3s-PMOD/parts/VGA/3D/DSUB-15-HD_Female_Horizontal_P2.29x1.98mm_EdgePinOffset3.03mm_Housed_MountingHolesOffset4.94mm.step
       (at (xyz 0 0 0))
@@
       (xy -4.18592 -1.25984) (xy -4.151381 -1.25984) (xy -4.130649 -1.261396)) (layer B.SilkS) (width 0.01))
   )
-  (gr_text V_1.0 (at 104.61 53.16 90) (layer F.SilkS)
+  (gr_text V_1.1 (at 104.61 53.16 90) (layer F.SilkS)
     (effects (font (size 1.5 1.5) (thickness 0.3)))
   )
