File: GPDI_ULX3S/GPDI_ULX3S.sch (KiCad schematic (older format))
At the start: 47 parts, among them J2 CONN, P1 GPDI, U1 RN5RK501A, U2 PCA9306

Commit message: GPDI update to KiCad 7, update PCA9306 package, Version to v1.6
Parts:
- D3: symbol GPDI_ULX3S_PMOD-rescue:D_Zener_Small-antena-GPDI_ULX3S_PMOD-rescue -> Device:D_Zener_Small
- R10, R11, R12, R13, R14, R15, R16, R17, R18, R19, R20, R21, R22, R23, R8, R9: symbol GPDI_ULX3S_PMOD-rescue:R-antena-GPDI_ULX3S_PMOD-rescue -> Device:R
Changed lines of the file:
@@
 CLK-
 $Comp
-L GPDI_ULX3S_PMOD-rescue:R-antena-GPDI_ULX3S_PMOD-rescue R11
+L Device:R R11
 U 1 1 5E2CBDF3
 P 4500 1800
@@
 $EndComp
 $Comp
-L GPDI_ULX3S_PMOD-rescue:R-antena-GPDI_ULX3S_PMOD-rescue R12
+L Device:R R12
 U 1 1 5E2CC017
 P 4700 1800
@@
 $EndComp
 $Comp
-L GPDI_ULX3S_PMOD-rescue:R-antena-GPDI_ULX3S_PMOD-rescue R15
+L Device:R R15
 U 1 1 5E2CC065
 P 4900 1800
@@
 $EndComp
 $Comp
-L GPDI_ULX3S_PMOD-rescue:R-antena-GPDI_ULX3S_PMOD-rescue R16
+L Device:R R16
 U 1 1 5E2CC0C5
 P 5100 1800
@@
 $EndComp
 $Comp
-L GPDI_ULX3S_PMOD-rescue:R-antena-GPDI_ULX3S_PMOD-rescue R19
+L Device:R R19
 U 1 1 5E2CC11B
 P 5300 1800
@@
 $EndComp
 $Comp
-L GPDI_ULX3S_PMOD-rescue:R-antena-GPDI_ULX3S_PMOD-rescue R20
+L Device:R R20
 U 1 1 5E2CC16F
 P 5500 1800
@@
 $EndComp
 $Comp
-L GPDI_ULX3S_PMOD-rescue:R-antena-GPDI_ULX3S_PMOD-rescue R8
+L Device:R R8
 U 1 1 5E2CC1C5
 P 4300 1800
@@
 $EndComp
 $Comp
-L GPDI_ULX3S_PMOD-rescue:R-antena-GPDI_ULX3S_PMOD-rescue R23
+L Device:R R23
 U 1 1 5E2CC21D
 P 5700 1800
@@
 $EndComp
 $Comp
-L GPDI_ULX3S_PMOD-rescue:R-antena-GPDI_ULX3S_PMOD-rescue R17
+L Device:R R17
 U 1 1 5E34419C
 P 7100 1350
@@
 $EndComp
 $Comp
-L GPDI_ULX3S_PMOD-rescue:R-antena-GPDI_ULX3S_PMOD-rescue R18
+L Device:R R18
 U 1 1 5E3441A2
 P 7100 1800
@@
 GPDI_D2+
 $Comp
-L GPDI_ULX3S_PMOD-rescue:R-antena-GPDI_ULX3S_PMOD-rescue R13
+L Device:R R13
 U 1 1 5E34947B
 P 6600 1350
@@
 $EndComp
 $Comp
-L GPDI_ULX3S_PMOD-rescue:R-antena-GPDI_ULX3S_PMOD-rescue R14
+L Device:R R14
 U 1 1 5E349481
 P 6600 1800
@@
 GPDI_D1+
 $Comp
-L GPDI_ULX3S_PMOD-rescue:R-antena-GPDI_ULX3S_PMOD-rescue R9
+L Device:R R9
 U 1 1 5E34949B
 P 6150 1350
@@
 $EndComp
 $Comp
-L GPDI_ULX3S_PMOD-rescue:R-antena-GPDI_ULX3S_PMOD-rescue R10
+L Device:R R10
 U 1 1 5E3494A1
 P 6150 1800
@@
 $EndComp
 $Comp
-L GPDI_ULX3S_PMOD-rescue:R-antena-GPDI_ULX3S_PMOD-rescue R22
+L Device:R R22
 U 1 1 5E316F15
 P 7550 1800
@@
 $EndComp
 $Comp
-L GPDI_ULX3S_PMOD-rescue:R-antena-GPDI_ULX3S_PMOD-rescue R21
+L Device:R R21
 U 1 1 5E316EA7
 P 7550 1350
@@
 	7550 1950 7550 2050
 $Comp
-L GPDI_ULX3S_PMOD-rescue:D_Zener_Small-antena-GPDI_ULX3S_PMOD-rescue D3
+L Device:D_Zener_Small D3
 U 1 1 5F5539A7
 P 10300 4300
